File: Blinky/Blinky_01_Layout/Blinky.kicad_pcb (KiCad board)
At the start: 2 copper layers, 0 parts

Commit message: Added the default edge cut
Other:
- board outline added: 29 x 29 mm
Changed lines of the file:
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@@
-(kicad_pcb (version 20171130) (host pcbnew "(5.0.0)")
+(kicad_pcb (version 20171130) (host pcbnew "(5.0.1-3-g963ef8bb5)")
   (general
     (thickness 1.6)
-    (drawings 0)
+    (drawings 8)
     (tracks 0)
     (zones 0)
@@
     (pad_drill 0.762)
     (pad_to_mask_clearance 0)
+    (solder_mask_min_width 0.25)
     (aux_axis_origin 0 0)
     (visible_elements 7FFFFFFF)
@@
     (uvia_drill 0.1)
   )
+  (gr_line (start 122 65) (end 134 65) (layer Edge.Cuts) (width 0.15))
+  (gr_line (start 134 65) (end 142.5 73.5) (layer Edge.Cuts) (width 0.15))
+  (gr_line (start 142.5 73.5) (end 142.5 85.5) (layer Edge.Cuts) (width 0.15))
+  (gr_line (start 142.5 85.5) (end 134 94) (layer Edge.Cuts) (width 0.15))
+  (gr_line (start 134 94) (end 122 94) (layer Edge.Cuts) (width 0.15))
+  (gr_line (start 122 94) (end 113.5 85.5) (layer Edge.Cuts) (width 0.15))
+  (gr_line (start 113.5 85.5) (end 113.5 73.5) (layer Edge.Cuts) (width 0.15))
+  (gr_line (start 113.5 73.5) (end 122 65) (layer Edge.Cuts) (width 0.15))
 )

Commit message: Removed the octagonal edge cut
Other:
- board outline removed
Changed lines of the file:
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@@
   (general
     (thickness 1.6)
-    (drawings 8)
+    (drawings 0)
     (tracks 0)
     (zones 0)
@@
     (uvia_drill 0.1)
   )
-  (gr_line (start 122 65) (end 134 65) (layer Edge.Cuts) (width 0.15))
-  (gr_line (start 134 65) (end 142.5 73.5) (layer Edge.Cuts) (width 0.15))
-  (gr_line (start 142.5 73.5) (end 142.5 85.5) (layer Edge.Cuts) (width 0.15))
-  (gr_line (start 142.5 85.5) (end 134 94) (layer Edge.Cuts) (width 0.15))
-  (gr_line (start 134 94) (end 122 94) (layer Edge.Cuts) (width 0.15))
-  (gr_line (start 122 94) (end 113.5 85.5) (layer Edge.Cuts) (width 0.15))
-  (gr_line (start 113.5 85.5) (end 113.5 73.5) (layer Edge.Cuts) (width 0.15))
-  (gr_line (start 113.5 73.5) (end 122 65) (layer Edge.Cuts) (width 0.15))
 )
