File: Blinky/Blinky_03_Layout/Blinky.kicad_pcb (KiCad board)
At the start: 2 copper layers, 29 x 29 mm, 12 parts, among them SW1 SW_SPDT, U1 NE555

Commit message: 03 Layout partially done
Parts:
- removed C3: 300n, Capacitors_SMD:C_0805
- removed REF***: KiCad-Logo2_6mm_SilkScreen, Symbols:KiCad-Logo2_6mm_SilkScreen
- added C1: 300n, Capacitor_SMD:C_0805_2012Metric, F.Cu at (70.5, 83.4)
- C2: footprint Capacitors_SMD:C_0805 -> Capacitor_SMD:C_0805_2012Metric
- D1, D2: footprint LEDs:LED_0805 -> LED_SMD:LED_0805_2012Metric
- R1, R4: footprint Resistors_SMD:R_0805 -> Resistor_SMD:R_0805_2012Metric
- R2: value 200 -> 1M; footprint Resistors_SMD:R_0805 -> Resistor_SMD:R_0805_2012Metric
- R3: value 1M -> 200; footprint Resistors_SMD:R_0805 -> Resistor_SMD:R_0805_2012Metric
- SW1: footprint Blinky:Micro_Schiebeschalter -> Button_Switch_SMD:SW_SPDT_PCM12
- U1: footprint Housings_SOIC:SOIC-8_3.9x4.9mm_Pitch1.27mm -> Package_SO:SOIC-8_3.9x4.9mm_P1.27mm
- moved D2 22.2 mm to (80.0, 93.3), turned to 270 degrees
- moved R4 21.8 mm to (80.0, 89.3), turned to 90 degrees
- moved D1 20.6 mm to (60.5, 93.3), turned to 270 degrees
- moved R3 14.4 mm to (60.5, 89.3), turned to 90 degrees
- moved R2 7.15 mm to (76.5, 86.6)
- moved C2 6.55 mm to (70.2, 92.1), turned to 0 degrees
- moved R1 2.38 mm to (76.5, 82.8)
- moved BT1 1.72 mm to (70.3, 87.9)
- moved U1 1.70 mm to (70.0, 87.9)
- moved SW1 0.71 mm to (69.5, 101.5), turned to 180 degrees
Connections:
- R2 pad 1: Net-(D1-Pad1) -> Net-(R1-Pad2)
- R2 pad 2: Net-(D2-Pad2) -> Net-(C1-Pad1)
- R3 pad 1: Net-(R1-Pad2) -> Net-(D1-Pad1)
- R3 pad 2: Net-(C3-Pad1) -> Net-(D2-Pad2)
- U1 pad 2: Net-(C3-Pad1) -> Net-(C1-Pad1)
- U1 pad 6: Net-(C3-Pad1) -> Net-(C1-Pad1)
Routing:
- net Net-(D2-Pad2): track 25.4 -> 0.00 mm
- net Net-(C3-Pad1): track 13.0 -> 0.00 mm
- net Net-(C1-Pad1): track 0.00 -> 9.42 mm
- net Net-(BT1-Pad1): track 25.3 -> 31.0 mm
- net /Vcc: track 8.98 -> 13.8 mm, vias 4 -> 2
- net GND: track 2.64 -> 0.00 mm, vias 1 -> 0
- net Net-(R1-Pad2): track 4.88 -> 6.34 mm
Other:
- board text removed: "Blinky Rev 2"
