File: Blinky/Blinky_02_Layout/Blinky.kicad_pcb (KiCad board)
At the start: 2 copper layers, 29 x 29 mm, 11 parts, among them SW1 SW_SPDT, U1 NE555

Commit message: Refit for Windows
Parts:
- removed C3: 300n, Capacitors_SMD:C_0805
- added C1: 300n, Capacitor_SMD:C_0805_2012Metric, F.Cu at (69.9, 85.8)
- C2: footprint Capacitors_SMD:C_0805 -> Capacitor_SMD:C_0805_2012Metric
- D1, D2: footprint LEDs:LED_0805 -> LED_SMD:LED_0805_2012Metric
- R1, R4: footprint Resistors_SMD:R_0805 -> Resistor_SMD:R_0805_2012Metric
- R2: value 200 -> 1M; footprint Resistors_SMD:R_0805 -> Resistor_SMD:R_0805_2012Metric
- R3: value 1M -> 200; footprint Resistors_SMD:R_0805 -> Resistor_SMD:R_0805_2012Metric
- SW1: footprint Blinky:Micro_Schiebeschalter -> Button_Switch_SMD:SW_SPDT_PCM12
- U1: footprint Housings_SOIC:SOIC-8_3.9x4.9mm_Pitch1.27mm -> Package_SO:SOIC-8_3.9x4.9mm_P1.27mm
- moved D2 22.3 mm to (80.0, 93.9), turned to 270 degrees
- moved R4 21.8 mm to (80.0, 89.7), turned to 90 degrees
- moved D1 21.6 mm to (59.6, 94.0), turned to 270 degrees
- moved R3 15.5 mm to (59.5, 89.8), turned to 90 degrees
- moved R2 7.38 mm to (74.9, 87.6)
- moved C2 5.84 mm to (64.8, 89.1), turned to 90 degrees
- moved SW1 0.94 mm to (69.8, 101.6), turned to 180 degrees
- moved R1 0.82 mm to (74.8, 83.7)
- moved U1 0.68 mm to (69.8, 90.2)
- moved BT1 0.64 mm to (69.9, 89.9)
Connections:
- R2 pad 1: Net-(D1-Pad1) -> Net-(R1-Pad2)
- R2 pad 2: Net-(D2-Pad2) -> Net-(C1-Pad1)
- R3 pad 1: Net-(R1-Pad2) -> Net-(D1-Pad1)
- R3 pad 2: Net-(C3-Pad1) -> Net-(D2-Pad2)
- U1 pad 2: Net-(C3-Pad1) -> Net-(C1-Pad1)
- U1 pad 6: Net-(C3-Pad1) -> Net-(C1-Pad1)
